Commit message: final for manuel ackerman steering controller

File: urdf/car_urdf.urdf (robot description, URDF)
Before this commit: robot car_urdf, 8 links, 7 joints
Links:
- removed link world
- added link dummy
- link rr_wheel: mass 0 -> 0.015904
Joints:
- removed joint base_joint
- removed joint fl_wheeel_j
- added joint dummy_joint: type fixed, parent dummy, child base_link, origin xyz=0.0 0.0 0.0 rpy=0 0 0
- added joint fl_wheel_j: type continuous, parent fl_pin, child fl_wheel, origin xyz=0 0.005 -0.004 rpy=0 0 0, axis 0 1 0, limit effort=200 velocity=30
- joint fl_pin_j: limit lower=-0.6 upper=0.6 effort=0 velocity=0 -> lower=-0.6 upper=0.6 effort=200 velocity=30; origin xyz=0 0 0 rpy=0 0 0 -> xyz=0.065223 0.045 0.004 rpy=0 0 0
- joint fr_pin_j: limit lower=-0.6 upper=0.6 effort=0 velocity=0 -> lower=-0.6 upper=0.6 effort=200 velocity=30
- joint fr_wheel_j: axis 0 -1 0 -> 0 1 0; limit (none) -> effort=200 velocity=30
- joint rl_wheel_j: axis 0 -1 0 -> 0 1 0; limit (none) -> effort=200 velocity=30
- joint rr_wheel_j: limit (none) -> effort=200 velocity=30
